File: test-projects/warning-project/warning-project.sch (KiCad schematic (older format))
At the start: 3 parts, among them J1 Conn_01x02

Commit message: Update test projects to KiCad 5
Parts:
- D1: symbol LED -> Device:LED
- J1: symbol Conn_01x02 -> Connector_Generic:Conn_01x02
- R1: symbol R -> Device:R
Connections:
- wire segments 8 -> 10
Changed lines of the file:
@@
-EESchema Schematic File Version 2
-LIBS:power
-LIBS:device
-LIBS:transistors
-LIBS:conn
-LIBS:linear
-LIBS:regul
-LIBS:74xx
-LIBS:cmos4000
-LIBS:adc-dac
-LIBS:memory
-LIBS:xilinx
-LIBS:microcontrollers
-LIBS:dsp
-LIBS:microchip
-LIBS:analog_switches
-LIBS:motorola
-LIBS:texas
-LIBS:intel
-LIBS:audio
-LIBS:interface
-LIBS:digital-audio
-LIBS:philips
-LIBS:display
-LIBS:cypress
-LIBS:siliconi
-LIBS:opto
-LIBS:atmel
-LIBS:contrib
-LIBS:valves
+EESchema Schematic File Version 4
 LIBS:warning-project-cache
-EELAYER 25 0
+EELAYER 26 0
 EELAYER END
 $Descr A4 11693 8268
@@
 $EndDescr
 $Comp
-L R R1
+L Device:R R1
 U 1 1 5CA32696
 P 3100 3425
@@
 $EndComp
 $Comp
-L LED D1
+L Device:LED D1
 U 1 1 5CA326B7
 P 3100 3075
@@
 $EndComp
 $Comp
-L VCC #PWR01
+L power:VCC #PWR01
 U 1 1 5CA32709
 P 3100 2875
@@
 $EndComp
 $Comp
-L Conn_01x02 J1
+L Connector_Generic:Conn_01x02 J1
 U 1 1 5CA32731
 P 2000 3125
@@
 $EndComp
 $Comp
-L VCC #PWR02
+L power:VCC #PWR02
 U 1 1 5CA327B9
 P 2625 2875
@@
 $EndComp
 $Comp
-L GND #PWR03
+L power:GND #PWR03
 U 1 1 5CA32803
 P 2625 3250
@@
 $EndComp
 $Comp
-L PWR_FLAG #FLG04
+L power:PWR_FLAG #FLG04
 U 1 1 5CA341D3
 P 2300 3250
@@
 $EndComp
 $Comp
-L GND #PWR05
+L power:GND #PWR05
 U 1 1 5CA38687
 P 3100 3650
@@
 $EndComp
 Wire Wire Line
-	2200 3025 2625 3025
+	2200 3025 2300 3025
 Wire Wire Line
 	3100 2875 3100 2925
 Wire Wire Line
-	2200 3125 2625 3125
+	2200 3125 2300 3125
 Wire Wire Line
 	2625 3025 2625 2875
@@
 Wire Wire Line
 	3100 3225 3100 3275
+Wire Wire Line
+	2300 3025 2625 3025
+Wire Wire Line
+	2300 3125 2625 3125
 $EndSCHEMATC
